Commit message: [planning] add obstacle model and modify iris_region_from_clique_builder to set obstacle pose from plant information

File: planning/2d_arms/box_small_with_obstacle.urdf (robot description, URDF)
Before this commit: robot box_scene, 6 links, 5 joints
Links:
- link box_obs: geometry collision box size=0.2 0.2 0.2; visual box size=0.2 0.2 0.2
